File: MCU Data Logger.kicad_sch (KiCad schematic)
At the start: 0 parts

Commit message: all required symbols
Parts:
- added BT?: Battery, symbol Device:Battery
- added C? (x4): C, symbol Device:C
- added C?: C_Polarized, symbol Device:C_Polarized
- added D? (x2): LED, symbol Device:LED
- added H? (x4): MountingHole, symbol Mechanical:MountingHole
- added R? (x7): R, symbol Device:R
- added U? (x2): 24LC1025, symbol Memory_EEPROM:24LC1025
- added U?: ATmega328P-A, Package_QFP:TQFP-32_7x7mm_P0.8mm, symbol MCU_Microchip_ATmega:ATmega328P-A
- added U?: DS1337S_, DS1337S_:SOIC127P600X175-8N, symbol DS1337S_:DS1337S_
- added Y? (x2): Crystal, symbol Device:Crystal
Connections:
- new net: U?.21 (GND), U?.3 (GND), U?.5 (GND)
- new net: U?.4 (VCC), U?.6 (VCC)
- new net: Y?.1, Y?.2
Other:
- added sheet Connectors (connectors.kicad_sch)
- company: (none) -> Primzel Technologies
- title: (none) -> MCU Data Logger

Commit message: updated values
Parts:
- C1, C2: renamed from C?; value C -> 0.1uF
- C3, C4: renamed from C?; value C -> 22pF
- C5: renamed from C?; value C_Polarized -> 100nF
- R1, R2: renamed from R?; value R -> 4.7K
- R3, R4, R5: renamed from R?; value R -> 10K
- R6, R7: renamed from R?; value R -> 330
- Y1: renamed from Y?; value Crystal -> 32.768KHz
- Y2: renamed from Y?; footprint (none) -> 16MHz
- gave numbers to parts that had none: 11
Connections:
- net at Y2.1: no longer Y1.2
Other:
- moved on the sheet: BT1, C1, C2, C3, C4, C5, D1, D2, H1, H2, H3, H4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

Commit message: wiring complete
Parts:
- BT1: footprint (none) -> Connector_PinHeader_2.54mm:PinHeader_1x02_P2.54mm_Vertical
- C1, C2, C3, C4, C5: footprint (none) -> Capacitor_SMD:C_0805_2012Metric
- D1, D2: footprint (none) -> LED_SMD:LED_0805_2012Metric
- H1, H2, H3, H4: footprint (none) -> MountingHole:MountingHole_2.1mm
- R1, R2, R3, R4, R5, R6, R7: footprint (none) -> Resistor_SMD:R_0805_2012Metric
- U1, U2: footprint (none) -> Package_SO:SOIC-8_5.3x5.3mm_P1.27mm
- U3: footprint DS1337S_:SOIC127P600X175-8N -> DS1337S:SOIC127P600X175-8N
- U4: footprint Package_QFP:TQFP-32_7x7mm_P0.8mm -> Package_QFP:LQFP-32_7x7mm_P0.8mm
- Y1: footprint (none) -> Crystal:Crystal_SMD_5032-2Pin_5.0x3.2mm
- Y2: value Crystal -> 16MHz; footprint 16MHz -> Crystal:Crystal_SMD_5032-2Pin_5.0x3.2mm
Connections:
- net Vcc: now reaches U2.1 (A0)
- net Vcc: now also C2.1, R1.1, R2.1, R3.1, R4.1, R5.1, U1.1 (A0), U1.2 (A1), U1.3 (A2), U1.8 (VCC), U2.3 (A2), U2.8 (VCC), U3.8 (VCC)
- net GND: now reaches U2.2 (A1)
- net GND: now also BT1.2 (-), C1.2, C2.2, C3.2, C4.1, C5.2, R6.1, R7.1, U1.4 (GND), U1.7 (WP), U2.4 (GND), U2.7 (WP), U3.4 (GND), U4.21 (GND), U4.3 (GND), U4.5 (GND)
- net SDA: now reaches U2.5 (SDA)
- net SDA: now also R2.2, U1.5 (SDA), U3.5 (SDA), U4.27 (PC4)
- net SCK: now reaches U2.6 (SCL)
- net SCK: now also D1.2 (A), R1.2, U1.6 (SCL), U3.6 (SCL), U4.17 (PB5), U4.28 (PC5)
- net at BT1.1 (+): now also C5.1, D2.2 (A), U4.18 (AVCC), U4.4 (VCC), U4.6 (VCC)
- net D3: now reaches U4.1 (PD3)
- net D6: now reaches U4.10 (PD6)
- net D7: now reaches U4.11 (PD7)
- net D8: now reaches U4.12 (PB0)
- net MOSI: now reaches U4.15 (PB3)
- net MISO: now reaches U4.16 (PB4)
- net D4: now reaches U4.2 (PD4)
- net at U4.20 (AREF): now also C1.1
- net RESET: now reaches U4.29 (~{RESET}/PC6)
- net RESET: now also R3.2
- net RX: now reaches U4.30 (PD0)
- net TX: now reaches U4.31 (PD1)
- net D2: now reaches U4.32 (PD2)
- net at U4.7 (XTAL1/PB6): now also C3.1, Y2.2
- net at U4.8 (XTAL2/PB7): now also C4.2, Y2.1
- net D5: now reaches U4.9 (PD5)
- net at D2.1 (K): now also R6.2
- net at R4.2: now also U3.7 (SQW/~INT)
- net at D1.1 (K): now also R7.2
- net at Y1.1: now also U3.2 (X2)
- net at Y1.2: now also U3.1 (X1)
- net at U3.3 (~{INTA}): now also R5.2
- no-connect marks 0 -> 8
Other:
- sheet Connectors ports: added D2, D3, D4, D5, D6, D7, D8, GND, MISO, MOSI, RESET, RX, SCK, SDA, TX, Vcc; removed none
- moved on the sheet: BT1, C1, C3, C4, C5, D1, D2, R3, R6, R7, U4, Y2
