File: MCU Data Logger.kicad_sch (KiCad schematic)
At the start: 25 parts, among them U1 24LC1025, U2 24LC1025, U3 DS1337S_, U4 ATmega328P-A, Y1 32.768KHz, Y2 16MHz

Commit message: complete PCB
Other:
- moved on the sheet: BT1, C1, C3, C4, C5, D1, D2, R3, R6, R7, U4, Y2

Commit message: bug fix
Connections:
- net SCK: no longer R1.2, U1.6 (SCL), U2.6 (SCL), U3.6 (SCL), U4.28 (PC5)
- new net SCL: R1.2, U1.6 (SCL), U2.6 (SCL), U3.6 (SCL), U4.28 (PC5)
Other:
- sheet Connectors ports: added SCL; removed none
Changed lines of the file:
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@@
 	(wire
 		(pts
-			(xy 207.01 135.89) (xy 217.17 135.89)
-		)
-		(stroke
-			(width 0)
-			(type default)
-		)
-	)
-	(wire
-		(pts
 			(xy 195.58 27.94) (xy 207.01 27.94)
 		)
@@
 	(wire
 		(pts
+			(xy 217.17 137.16) (xy 224.79 137.16)
+		)
+		(stroke
+			(width 0)
+			(type default)
+		)
+	)
+	(wire
+		(pts
 			(xy 17.78 57.15) (xy 27.94 57.15)
 		)
@@
 	(wire
 		(pts
-			(xy 63.5 62.23) (xy 68.58 62.23)
+			(xy 195.58 154.94) (xy 224.79 154.94)
 		)
 		(stroke
@@
 	(wire
 		(pts
-			(xy 68.58 62.23) (xy 68.58 69.85)
+			(xy 63.5 62.23) (xy 68.58 62.23)
 		)
 		(stroke
@@
 	(wire
 		(pts
-			(xy 201.93 80.01) (xy 209.55 80.01)
+			(xy 68.58 62.23) (xy 68.58 69.85)
 		)
 		(stroke
@@
 	(wire
 		(pts
-			(xy 196.85 139.7) (xy 224.79 139.7)
+			(xy 201.93 80.01) (xy 209.55 80.01)
 		)
 		(stroke
@@
 	(wire
 		(pts
-			(xy 91.44 157.48) (xy 91.44 161.29)
+			(xy 196.85 139.7) (xy 224.79 139.7)
 		)
 		(stroke
@@
 	(wire
 		(pts
-			(xy 191.77 36.83) (xy 191.77 39.37)
+			(xy 91.44 157.48) (xy 91.44 161.29)
 		)
 		(stroke
@@
 	(wire
 		(pts
-			(xy 207.01 135.89) (xy 207.01 137.16)
+			(xy 191.77 36.83) (xy 191.77 39.37)
 		)
 		(stroke
@@
 	(wire
 		(pts
-			(xy 207.01 137.16) (xy 224.79 137.16)
-		)
-		(stroke
-			(width 0)
-			(type default)
-		)
-	)
-	(wire
-		(pts
 			(xy 17.78 55.88) (xy 17.78 57.15)
 		)
@@
 	(wire
 		(pts
+			(xy 88.9 30.48) (xy 88.9 34.29)
+		)
+		(stroke
+			(width 0)
+			(type default)
+		)
+	)
+	(wire
+		(pts
 			(xy 91.44 172.72) (xy 91.44 168.91)
 		)
@@
 	(wire
 		(pts
+			(xy 217.17 135.89) (xy 217.17 137.16)
+		)
+		(stroke
+			(width 0)
+			(type default)
+		)
+	)
+	(wire
+		(pts
 			(xy 76.2 34.29) (xy 85.09 34.29)
 		)
@@
 		)
 	)
-	(label "SCK"
-		(at 196.85 146.05 180)
-		(effects
-			(font
-				(size 1.27 1.27)
-			)
-			(justify right bottom)
-		)
-	)
 	(label "D5"
 		(at 210.82 99.06 180)
@@
 		)
 	)
+	(label "SCK"
+		(at 195.58 154.94 180)
+		(effects
+			(font
+				(size 1.27 1.27)
+			)
+			(justify right bottom)
+		)
+	)
 	(label "SDA"
 		(at 49.53 163.83 0)
@@
 		)
 	)
-	(label "SCK"
+	(label "SCL"
 		(at 210.82 78.74 180)
 		(effects
@@
 		)
 	)
-	(label "SCK"
-		(at 85.09 171.45 180)
-		(effects
-			(font
-				(size 1.27 1.27)
-			)
-			(justify right bottom)
-		)
-	)
 	(label "D7"
 		(at 210.82 104.14 180)
@@
 		)
 	)
+	(label "SCL"
+		(at 74.93 166.37 0)
+		(effects
+			(font
+				(size 1.27 1.27)
+			)
+			(justify left bottom)
+		)
+	)
 	(label "D3"
 		(at 210.82 93.98 180)
@@
 		)
 	)
+	(label "SCL"
+		(at 85.09 171.45 0)
+		(effects
+			(font
+				(size 1.27 1.27)
+			)
+			(justify left bottom)
+		)
+	)
 	(label "MOSI"
 		(at 210.82 50.8 180)
@@
 	)
 	(label "RESET"
-		(at 205.74 80.01 0)
+		(at 201.93 80.01 0)
 		(effects
 			(font
@@
 		)
 	)
+	(label "SCL"
+		(at 196.85 146.05 180)
+		(effects
+			(font
+				(size 1.27 1.27)
+			)
+			(justify right bottom)
+		)
+	)
 	(label "D6"
 		(at 210.82 101.6 180)
@@
 		)
 	)
-	(label "SCK"
-		(at 49.53 166.37 0)
-		(effects
-			(font
-				(size 1.27 1.27)
-			)
-			(justify left bottom)
-		)
-	)
 	(label "RESET"
 		(at 208.28 162.56 180)
@@
 		)
 	)
-	(label "SCK"
-		(at 74.93 166.37 0)
-		(effects
-			(font
-				(size 1.27 1.27)
-			)
-			(justify left bottom)
-		)
-	)
 	(label "D3"
 		(at 237.49 143.51 0)
@@
 		)
 	)
-	(label "SCK"
+	(label "SCL"
 		(at 27.94 44.45 180)
 		(effects
@@
 		)
 	)
+	(label "SCL"
+		(at 49.53 166.37 0)
+		(effects
+			(font
+				(size 1.27 1.27)
+			)
+			(justify left bottom)
+		)
+	)
 	(label "D8"
 		(at 210.82 43.18 180)
@@
 	(symbol
 		(lib_id "power:PWR_FLAG")
-		(at 88.9 34.29 0)
+		(at 88.9 30.48 0)
 		(unit 1)
 		(exclude_from_sim no)
@@
 		(fields_autoplaced yes)
 		(property "Reference" "#FLG03"
-			(at 88.9 32.385 0)
+			(at 88.9 28.575 0)
 			(effects
 				(font
@@
 		)
 		(property "Value" "PWR_FLAG"
-			(at 88.9 29.21 0)
+			(at 88.9 25.4 0)
 			(effects
 				(font
@@
 		)
 		(property "Footprint" ""
-			(at 88.9 34.29 0)
+			(at 88.9 30.48 0)
 			(effects
 				(font
@@
 		)
 		(property "Datasheet" "~"
-			(at 88.9 34.29 0)
+			(at 88.9 30.48 0)
 			(effects
 				(font
@@
 		)
 		(property "Description" "Special symbol for telling ERC where power comes from"
-			(at 88.9 34.29 0)
+			(at 88.9 30.48 0)
+			(effects
+				(font
+					(size 1.27 1.27)
+				)
+				(hide yes)
+			)
+		)
+		(property "Purpose" ""
+			(at 88.9 30.48 0)
 			(effects
 				(font
@@
 			)
 		)
-		(pin "SCK" bidirectional
-			(at 224.79 146.05 180)
-			(effects
-				(font
-					(size 1.27 1.27)
-				)
-				(justify left)
-			)
-		)
 		(pin "D8" bidirectional
 			(at 237.49 156.21 0)
@@
 			)
 		)
+		(pin "SCK" passive
+			(at 224.79 154.94 180)
+			(effects
+				(font
+					(size 1.27 1.27)
+				)
+				(justify left)
+			)
+		)
+		(pin "SCL" bidirectional
+			(at 224.79 146.05 180)
+			(effects
+				(font
+					(size 1.27 1.27)
+				)
+				(justify left)
+			)
+		)
