File: connectors.kicad_sch (KiCad schematic)
At the start: 4 parts

Commit message: updated values
Parts:
- gave numbers to parts that had none: 4
Changed lines of the file:
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@@
 		(dnp no)
 		(fields_autoplaced yes)
-		(property "Reference" "J?"
+		(property "Reference" "J4"
 			(at 87.63 110.49 0)
 			(effects
@@
 			(project ""
 				(path "/025bd588-c6d4-455a-8333-36896a0f0dbe/6ca9abbd-edb3-4d51-9ca4-f0d2029b8830"
-					(reference "J?")
+					(reference "J4")
 					(unit 1)
 				)
@@
 		(on_board yes)
 		(dnp no)
-		(property "Reference" "J?"
+		(property "Reference" "J1"
 			(at 52.705 67.31 0)
 			(effects
@@
 			(project ""
 				(path "/025bd588-c6d4-455a-8333-36896a0f0dbe/6ca9abbd-edb3-4d51-9ca4-f0d2029b8830"
-					(reference "J?")
+					(reference "J1")
 					(unit 1)
 				)
@@
 		(dnp no)
 		(fields_autoplaced yes)
-		(property "Reference" "J?"
+		(property "Reference" "J2"
 			(at 52.705 101.6 0)
 			(effects
@@
 			(project ""
 				(path "/025bd588-c6d4-455a-8333-36896a0f0dbe/6ca9abbd-edb3-4d51-9ca4-f0d2029b8830"
-					(reference "J?")
+					(reference "J2")
 					(unit 1)
 				)
@@
 		(on_board yes)
 		(dnp no)
-		(property "Reference" "J?"
+		(property "Reference" "J3"
 			(at 53.975 82.55 0)
 			(effects
@@
 			(project "MCU Data Logger"
 				(path "/025bd588-c6d4-455a-8333-36896a0f0dbe/6ca9abbd-edb3-4d51-9ca4-f0d2029b8830"
-					(reference "J?")
+					(reference "J3")
 					(unit 1)
 				)

Commit message: wiring complete
Parts:
- J1, J3: footprint (none) -> Connector_PinHeader_2.54mm:PinHeader_1x04_P2.54mm_Vertical
- J2: footprint (none) -> Connector_PinHeader_2.54mm:PinHeader_1x09_P2.54mm_Vertical
- J4: footprint (none) -> Connector_PinHeader_2.54mm:PinHeader_2x03_P2.54mm_Vertical
Connections:
- net MISO: now reaches J4.1 (Pin_1)
- net Vcc: now reaches J4.2 (Pin_2)
- net Vcc: now also J1.2 (Pin_2), J2.9 (Pin_9), J3.2 (Pin_2)
- net SCK: now reaches J4.3 (Pin_3)
- net SCK: now also J1.4 (Pin_4)
- net MOSI: now reaches J4.4 (Pin_4)
- net RESET: now reaches J4.5 (Pin_5)
- net GND: now reaches J4.6 (Pin_6)
- net GND: now also J1.1 (Pin_1), J2.8 (Pin_8), J3.1 (Pin_1)
- net SDA: now reaches J1.3 (Pin_3)
- net D2: now reaches J2.1 (Pin_1)
- net D3: now reaches J2.2 (Pin_2)
- net D4: now reaches J2.3 (Pin_3)
- net D5: now reaches J2.4 (Pin_4)
- net D6: now reaches J2.5 (Pin_5)
- net D7: now reaches J2.6 (Pin_6)
- net D8: now reaches J2.7 (Pin_7)
- net RX: now reaches J3.3 (Pin_3)
- net TX: now reaches J3.4 (Pin_4)
Other:
- moved on the sheet: J3

Commit message: bug fix
Connections:
- net SCK: no longer J1.4 (Pin_4)
- new net SCL: J1.4 (Pin_4)
Changed lines of the file:
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@@
 		)
 	)
-	(hierarchical_label "SCK"
+	(hierarchical_label "SCL"
 		(shape bidirectional)
 		(at 57.15 80.01 0)
