File: MCU Data Logger.kicad_pcb (KiCad board)
At the start: 2 copper layers, 79.1 x 49.1 mm, 28 parts, among them J1 Conn_01x04_Pin, J2 Conn_01x09_Pin, J3 Conn_01x04_Pin, J4 Conn_02x03_Odd_Even, U1 24LC1025, U2 24LC1025, U3 DS1337S_, U4 ATmega328P-A, Y1 32.768KHz, Y2 16MHz

Commit message: complete PCB
Parts:
- moved C4 23.2 mm to (114.3, 85.1), turned to 90 degrees
- moved C3 23.2 mm to (114.3, 81.3), turned to 90 degrees
Routing:
- net /Vcc: track 181.4 -> 18.4 mm, vias 5 -> 2
- net GND: track 61.5 -> 140.8 mm, vias 5 -> 9
- net Net-(U4-XTAL1/PB6): track 42.9 -> 17.5 mm
- net Net-(U4-XTAL2/PB7): track 43.2 -> 20.9 mm
- net Net-(BT1-+): track 44.9 -> 41.5 mm
- net /RX: track 45.1 -> 44.9 mm, vias 2 -> 1
- added copper zone on F.Cu, net /Vcc
- added copper zone on B.Cu, net GND
- removed copper zone on F.Cu, net GND

Commit message: bug fix
Parts:
- added R4: 10K, Resistor_SMD:R_0805_2012Metric, F.Cu at (105.4, 75.6)
Connections:
- J1 pad 4: /SCK -> /SCL
- R1 pad 2: /SCK -> /SCL
- U1 pad 6: /SCK -> /SCL
- U2 pad 6: /SCK -> /SCL
- U3 pad 6: /SCK -> /SCL
- U4 pad 28: /SCK -> /SCL
Routing:
- net /SCL: track 0.00 -> 79.6 mm, vias 0 -> 7
- net /SCK: track 128.5 -> 64.6 mm, vias 9 -> 2
- net /Vcc: track 18.4 -> 30.6 mm, vias 2 -> 4
- net Net-(U3-SQW/~INT): track 0.00 -> 5.38 mm
- net Net-(BT1-+): track 41.5 -> 41.9 mm, vias 0 -> 1
